File: tetrisBusinessCard/tetrisBusinessCard.kicad_pcb (KiCad board)
At the start: 2 copper layers, 48.7 x 84.5 mm, 499 parts, among them SW1 SW_Push, SW2 SW_Push, SW3 SW_Push, SW4 SW_Push, SW5 SW_Push, SW6 SW_Push, SW7 SW_DPST_x2, U1 SC091413, U2 W25Q16JVUXIQ, Y1 ABMB-272-T3

Commit message: update repo to be up to date with laptop backip
Parts:
- removed QR: LOGO, MyFootprints:qrCode
- B1: footprint MyFootprints:BAT_BS-02_MYG -> MyFootprints:BAT_BS-02_MYG-NoDrill
